File: Skeemid/Sammu-mootorite_skeem/Sammu-mootorite_skeem.kicad_sch (KiCad schematic)
At the start: 16 parts, among them SW2 SW_DPST_x2, SW4 SW_DPST_x2

Commit message: lisatud hultraheli andur
Parts:
- added U10: ~, symbol Tauno_Library:HC-SR04
Connections:
- net +5V: now also U10.1 (VCC)
- net GND: now also U10.4 (Gnd)
- new net D11: U10.2 (Trig)
- new net D12: U10.3 (Echo)
Other:
- note added: "Ultraheli andur HC-SR04"
- moved on the sheet: C1, C2, R3, R4, SW2A, SW4A

Commit message: Kolvi limit switch
Connections:
- net D11: now also A1.26 (D11)
- net D12: now also A1.27 (D12)
Other:
- note added: "Kolvi lüliti"
- note removed: "Vasakpoolne lüliti"
- moved on the sheet: U1, U2, U3, U4, U5

Commit message: pin reverse
Connections:
- net D7: now also C2.2, R4.1, SW4.2 (B); no longer C1.2, R3.1, SW2.2 (B)
- net D8: now also C1.2, R3.1, SW2.2 (B); no longer C2.2, R4.1, SW4.2 (B)
Changed lines of the file:
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@@
 		(title "Etteande skeem")
 		(date "2025-08-12")
-		(rev "1.2")
+		(rev "1.3")
 		(company "Tauno Erik")
 		(comment 1 "TSENTER")
@@
 		)
 	)
+	(label "D8"
+		(at 217.17 40.64 0)
+		(effects
+			(font
+				(size 1.27 1.27)
+			)
+			(justify left bottom)
+		)
+	)
 	(label "D7"
-		(at 217.17 40.64 0)
-		(effects
-			(font
-				(size 1.27 1.27)
-			)
-			(justify left bottom)
-		)
-	)
-	(label "D8"
 		(at 271.78 40.64 0)
 		(effects
