File: Kood/Juhtmoodul_KiCad/Juhtmoodul_skeem.kicad_sch (KiCad schematic)
At the start: 11 parts, among them SW2 SW_DPST_x2, U1 Pico moodul, U3 Andur, U4 Andur, U5 Andur

Commit message: juhtmooli sekeemi uuendused
Connections:
- net +3.3V: no longer U3.3 (IN), U4.3 (IN), U5.3 (IN)
- net +5V: no longer U1.10 (1_VCC), U1.5 (2_VCC), U2.1 (+5V), U7.2 (5V)
- net GND: now also U1.14 (GND), U3.4 (OUT), U4.4 (OUT), U5.4 (OUT)
- net GP15-Mootorite signaal: now also U1.8 (1_GND); no longer U1.3 (2_GND)
- net GP22-Silindri signaal: now also U1.3 (2_GND); no longer U1.8 (1_GND)
- net GP26-Andur_1_signaal: now also U3.3 (IN); no longer U3.4 (OUT)
- net GP27-Andur_2_signaal: now also U4.3 (IN); no longer U4.4 (OUT)
- net GP28-Andur_3_signaal: now also U5.3 (IN); no longer U5.4 (OUT)
- net at U1.4 (2_GPIO): now also U7.2 (5V)
- net at U1.9 (1_GPIO): now also U2.1 (+5V)
Other:
- moved on the sheet: C1, R3, SW2A, U1, U2, U3, U4, U5, U7, U8
